Commit message: Various clean up changes; added lidar simulation test

File: simulated_lidar_scanner/test/lidar_test.xacro (robot description, xacro)
@@ -6,13 +6,13 @@
     <visual>
       <geometry>
-        <mesh filename="package://lidar_scanner_node/test/view_object.stl"/>
+        <mesh filename="package://simulated_lidar_scanner/test/view_object.stl"/>
       </geometry>
       <material name="view_object_material">
-        <color rbga="0.8 0.8 0.8 1"/>
+        <color rbga="1 0 0 1"/>
       </material>
     </visual>
   </link>
   <joint name="lidar_parent_joint" type="fixed">
-    <origin xyz="0 0 0" rpy="0 0 0"/>
+    <origin xyz="1 0 2" rpy="0 -${radians(135)} 0"/>
     <parent link="odom"/>
     <child link="lidar_parent"/>
